Commit message: Make S20 a ur20-compatible macro

File: elfin_description/urdf/S20.urdf.xacro (robot description, xacro)
@@ -1,440 +1,454 @@
+<?xml version="1.0"?>
 <robot
   name="S20" xmlns:xacro="http://www.ros.org/wiki/xacro">
-  <xacro:include filename="$(find elfin_description)/urdf/materials.xacro" />
-  <xacro:include filename="$(find elfin_description)/urdf/elfin_robot.gazebo" />
-  <xacro:include filename="$(find elfin_description)/urdf/elfin_transmission.xacro" />
-  <xacro:property name="PI" value="3.1415926535897931"/>
-  <xacro:property name="density" value="3.09"/>
-  <link name="world"/>
-  <joint name="world_base" type="fixed">
-    <origin
-      xyz="0 0 0"
-      rpy="0 0 0" />
-    <parent
-      link="world" />
-    <child
-      link="elfin_base_link" />
-  </joint>
-  <link name="elfin_base_link"/>
-  <joint name="elfin_base_joint" type="fixed">
-    <origin
-      xyz="0 0 0"
-      rpy="0 0 0" />
-    <parent
-      link="elfin_base_link" />
-    <child
-      link="elfin_base" />
-  </joint>
-  <link
-    name="elfin_base">
-    <inertial>
-      <origin
-        xyz="-0.00131650768656017 3.86349405459754E-05 0.0343213199540785"
-        rpy="0 0 0" />
-      <mass
-        value="2.32181468230125" />
-      <inertia
-        ixx="0.00741739022505177"
-        ixy="-9.4225231258528E-05"
-        ixz="-5.45619950886553E-05"
-        iyy="0.00699483778046143"
-        iyz="1.30022773204213E-06"
-        izz="0.0123390065438587" />
-    </inertial>
-    <visual>
+  <xacro:macro name="s20" params="prefix:=elfin_ include_world:=true">
+    <xacro:include filename="$(find elfin_description)/urdf/materials.xacro" />
+    <xacro:include filename="$(find elfin_description)/urdf/elfin_robot.gazebo" />
+    <xacro:include filename="$(find elfin_description)/urdf/elfin_transmission.xacro" />
+    <xacro:property name="PI" value="3.1415926535897931"/>
+    <xacro:property name="density" value="3.09"/>
+    <!-- Used by Elfin S utilities -->
+    <xacro:if value="include_world">
+      <link name="world"/>
+      <joint name="world_base" type="fixed">
+        <origin
+          xyz="0 0 0"
+          rpy="0 0 0" />
+        <parent
+          link="world" />
+        <child
+          link="elfin_base_link" />
+      </joint>
+    </xacro:if>
+    <link name="${prefix}base_link"/>
+    <joint name="${prefix}base_joint" type="fixed">
       <origin
         xyz="0 0 0"
         rpy="0 0 0" />
-      <geometry>
-        <mesh
-          filename="package://elfin_description/meshes/S20/elfin_base.STL" />
-      </geometry>
-      <material
-        name="">
-        <color
-          rgba="0.752941176470588 0.752941176470588 0.752941176470588 1" />
-      </material>
-    </visual>
-    <collision>
-      <origin
-        xyz="0 0 0"
+      <parent
+        link="${prefix}base_link" />
+      <child
+        link="${prefix}base" />
+    </joint>
+    <link
+      name="${prefix}base">
+      <inertial>
+        <origin
+          xyz="-0.00131650768656017 3.86349405459754E-05 0.0343213199540785"
+          rpy="0 0 0" />
+        <mass
+          value="2.32181468230125" />
+        <inertia
+          ixx="0.00741739022505177"
+          ixy="-9.4225231258528E-05"
+          ixz="-5.45619950886553E-05"
+          iyy="0.00699483778046143"
+          iyz="1.30022773204213E-06"
+          izz="0.0123390065438587" />
+      </inertial>
+      <visual>
+        <origin
+          xyz="0 0 0"
+          rpy="0 0 0" />
+        <geometry>
+          <mesh
+            filename="package://elfin_description/meshes/S20/elfin_base.STL" />
+        </geometry>
+        <material
+          name="">
+          <color
+            rgba="0.752941176470588 0.752941176470588 0.752941176470588 1" />
+        </material>
+      </visual>
+      <collision>
+        <origin
+          xyz="0 0 0"
+          rpy="0 0 0" />
+        <geometry>
+          <mesh
+            filename="package://elfin_description/meshes/S20/elfin_base.STL" />
+        </geometry>
+      </collision>
+    </link>
+    <link
+      name="${prefix}shoulder_link">
+      <inertial>
+        <origin
+          xyz="-1.0792519167212E-07 -0.0224399626110038 0.00175002240516534"
+          rpy="0 0 0" />
+        <mass
+          value="6.93455742496729" />
+        <inertia
+          ixx="0.0460589183335357"
+          ixy="5.43718136375216E-07"
+          ixz="2.96738634298801E-07"
+          iyy="0.0375916708812216"
+          iyz="-0.000245581780149179"
+          izz="0.0394268304468804" />
+      </inertial>
+      <visual>
+        <origin
+          xyz="0 0 0"
+          rpy="0 0 0" />
+        <geometry>
+          <mesh
+            filename="package://elfin_description/meshes/S20/elfin_link1.STL" />
+        </geometry>
+        <material
+          name="">
+          <color
+            rgba="0.898039215686275 0.917647058823529 0.929411764705882 1" />
+        </material>
+      </visual>
+      <collision>
+        <origin
+          xyz="0 0 0"
+          rpy="0 0 0" />
+        <geometry>
+          <mesh
+            filename="package://elfin_description/meshes/S20/elfin_link1.STL" />
+        </geometry>
+      </collision>
+    </link>
+    <!-- shoulder_pan_joint -->
+    <joint
+      name="${prefix}shoulder_pan_joint"
+      type="revolute">
+      <origin
+        xyz="0 0 0.171"
         rpy="0 0 0" />
-      <geometry>
-        <mesh
-          filename="package://elfin_description/meshes/S20/elfin_base.STL" />
-      </geometry>
-    </collision>
-  </link>
-  <link
-    name="elfin_link1">
-    <inertial>
-      <origin
-        xyz="-1.0792519167212E-07 -0.0224399626110038 0.00175002240516534"
+      <parent
+        link="${prefix}base" />
+      <child
+        link="${prefix}shoulder_link" />
+      <axis
+        xyz="0 0 1" />
+    <limit
+        lower="-6.28"
+        upper="6.28"
+        effort="200"
+        velocity="1.57" />
+    </joint>
+    <link
+      name="${prefix}upper_arm_link">
+      <inertial>
+        <origin
+          xyz="-0.370229694350317 9.38128437405483E-07 0.000899041883029139"
+          rpy="0 0 0" />
+        <mass
+          value="18.8395085758056" />
+        <inertia
+          ixx="0.0687507132351259"
+          ixy="-5.05507420279161E-07"
+          ixz="-6.41343868263508E-05"
+          iyy="0.411200291693132"
+          iyz="-1.80729528146994E-07"
+          izz="0.40138597350588" />
+      </inertial>
+      <visual>
+        <origin
+          xyz="0 0 0"
+          rpy="0 0 0" />
+        <geometry>
+          <mesh
+            filename="package://elfin_description/meshes/S20/elfin_link2.STL" />
+        </geometry>
+        <material
+          name="">
+          <color
+            rgba="0.752941176470588 0.752941176470588 0.752941176470588 1" />
+        </material>
+      </visual>
+      <collision>
+        <origin
+          xyz="0 0 0"
+          rpy="0 0 0" />
+        <geometry>
+          <mesh
+            filename="package://elfin_description/meshes/S20/elfin_link2.STL" />
+        </geometry>
+      </collision>
+    </link>
+    <!-- shoulder_lift_joint -->
+    <joint
+      name="${prefix}shoulder_lift_joint"
+      type="revolute">
+      <origin
+        xyz="0 -0.2295 0"
+        rpy="1.5708 0 0" />
+      <parent
+        link="${prefix}shoulder_link" />
+      <child
+        link="${prefix}upper_arm_link" />
+      <axis
+        xyz="0 0 1" />
+      <limit
+        lower="-3.3158"
+        upper="0.1745"
+        effort="200"
+        velocity="1.57" />
+    </joint>
+    <link
+      name="${prefix}forearm_link">
+      <inertial>
+        <origin
+          xyz="0.310973076601113 -4.7405306624615E-09 0.0109938899740937"
+          rpy="0 0 0" />
+        <mass
+          value="7.53508270364931" />
+        <inertia
+          ixx="0.0133872719937165"
+          ixy="1.91460600478011E-07"
+          ixz="0.00152175061957157"
+          iyy="0.11837455186459"
+          iyz="-2.26041817837737E-08"
+          izz="0.116582348081593" />
+      </inertial>
+      <visual>
+        <origin
+          xyz="0 0 0"
+          rpy="0 0 0" />
+        <geometry>
+          <mesh
+            filename="package://elfin_description/meshes/S20/elfin_link3.STL" />
+        </geometry>
+        <material
+          name="">
+          <color
+            rgba="0.752941176470588 0.752941176470588 0.752941176470588 1" />
+        </material>
+      </visual>
+      <collision>
+        <origin
+          xyz="0 0 0"
+          rpy="0 0 0" />
+        <geometry>
+          <mesh
+            filename="package://elfin_description/meshes/S20/elfin_link3.STL" />
+        </geometry>
+      </collision>
+    </link>
+    <!-- elbow_joint -->
+    <joint
+      name="${prefix}elbow_joint"
+      type="revolute">
+      <origin
+        xyz="-0.85 0 -0.1885"
+        rpy="0 0 3.1416" />
+      <parent
+        link="${prefix}upper_arm_link" />
+      <child
+        link="${prefix}forearm_link" />
+      <axis
+        xyz="0 0 1" />
+      <limit
+        lower="-2.9319"
+        upper="2.9319"
+        effort="200"
+        velocity="1.57" />
+    </joint>
+    <link
+      name="${prefix}wrist_1_link">
+      <inertial>
+        <origin
+          xyz="8.5204157129759E-07 -0.00559612992738279 0.124499710924349"
+          rpy="0 0 0" />
+        <mass
+          value="1.26777180180805" />
+        <inertia
+          ixx="0.00300888445161096"
+          ixy="1.64612435809042E-08"
+          ixz="3.62281943568331E-08"
+          iyy="0.00214465218602862"
+          iyz="9.35786831203314E-05"
+          izz="0.00239761638151984" />
+      </inertial>
+      <visual>
+        <origin
+          xyz="0 0 0"
+          rpy="0 0 0" />
+        <geometry>
+          <mesh
+            filename="package://elfin_description/meshes/S20/elfin_link4.STL" />
+        </geometry>
+        <material
+          name="">
+          <color
+            rgba="0.898039215686275 0.917647058823529 0.929411764705882 1" />
+        </material>
+      </visual>
+      <collision>
+        <origin
+          xyz="0 0 0"
+          rpy="0 0 0" />
+        <geometry>
+          <mesh
+            filename="package://elfin_description/meshes/S20/elfin_link4.STL" />
+        </geometry>
+      </collision>
+    </link>
+    <!-- wrist_1_joint -->
+    <joint
+      name="${prefix}wrist_1_joint"
+      type="revolute">
+      <origin
+        xyz="0.712 0 0"
         rpy="0 0 0" />
-      <mass
-        value="6.93455742496729" />
-      <inertia
-        ixx="0.0460589183335357"
-        ixy="5.43718136375216E-07"
-        ixz="2.96738634298801E-07"
-        iyy="0.0375916708812216"
-        iyz="-0.000245581780149179"
-        izz="0.0394268304468804" />
-    </inertial>
-    <visual>
-      <origin
-        xyz="0 0 0"
-        rpy="0 0 0" />
-      <geometry>
-        <mesh
-          filename="package://elfin_description/meshes/S20/elfin_link1.STL" />
-      </geometry>
-      <material
-        name="">
-        <color
-          rgba="0.898039215686275 0.917647058823529 0.929411764705882 1" />
-      </material>
-    </visual>
-    <collision>
-      <origin
-        xyz="0 0 0"
-        rpy="0 0 0" />
-      <geometry>
-        <mesh
-          filename="package://elfin_description/meshes/S20/elfin_link1.STL" />
-      </geometry>
-    </collision>
-  </link>
-  <joint
-    name="elfin_joint1"
-    type="revolute">
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
Commit message: Fix a number of hard-coded values

File: elfin_description/urdf/S20.urdf.xacro (robot description, xacro)
@@ -1,6 +1,6 @@
-<?xml version="1.0"?>
+<?xml version="1.0" encoding="utf-8"?>
 <robot
   name="S20" xmlns:xacro="http://www.ros.org/wiki/xacro">
-  <xacro:macro name="s20" params="prefix:=elfin_ include_world:=true">
+  <xacro:macro name="S20" params="prefix:=elfin_ include_world:=true">
     <xacro:include filename="$(find elfin_description)/urdf/materials.xacro" />
     <xacro:include filename="$(find elfin_description)/urdf/elfin_robot.gazebo" />
@@ -9,5 +9,5 @@
     <xacro:property name="density" value="3.09"/>
     <!-- Used by Elfin S utilities -->
-    <xacro:if value="include_world">
+    <xacro:if value="${include_world}">
       <link name="world"/>
       <joint name="world_base" type="fixed">
@@ -18,5 +18,5 @@
           link="world" />
         <child
-          link="elfin_base_link" />
+          link="${prefix}base_link" />
       </joint>
     </xacro:if>

Commit message: Xacro fixup and move group hack

File: elfin_description/urdf/S20.urdf.xacro (robot description, xacro)
@@ -9,5 +9,5 @@
     <xacro:property name="density" value="3.09"/>
     <!-- Used by Elfin S utilities -->
-    <xacro:if value="include_world">
+    <xacro:if value="${include_world}">
       <link name="world"/>
       <joint name="world_base" type="fixed">
@@ -111,5 +111,4 @@
       </collision>
     </link>
-    <!-- shoulder_pan_joint -->
     <joint
       name="${prefix}shoulder_pan_joint"
@@ -170,5 +169,4 @@
       </collision>
     </link>
-    <!-- shoulder_lift_joint -->
     <joint
       name="${prefix}shoulder_lift_joint"
@@ -229,5 +227,4 @@
       </collision>
     </link>
-    <!-- elbow_joint -->
     <joint
       name="${prefix}elbow_joint"
@@ -288,5 +285,4 @@
       </collision>
     </link>
-    <!-- wrist_1_joint -->
     <joint
       name="${prefix}wrist_1_joint"
@@ -347,5 +343,4 @@
       </collision>
     </link>
-    <!-- wrist_2_joint -->
     <joint
       name="${prefix}wrist_2_joint"
@@ -406,6 +401,10 @@
       </collision>
     </link>
-    <!-- TODO: localization_joint is missing -->
-    <!-- wrist_3_joint -->
+    <link name="${prefix}localization_link" />
+    <joint name="${prefix}localization_joint" type="fixed">
+      <origin xyz="0 0 0.138" rpy="0 0 0" />
+      <parent link="${prefix}wrist_2_link" />
+      <child link="${prefix}localization_link" />
+    </joint>
     <joint
       name="${prefix}wrist_3_joint"
@@ -429,5 +428,4 @@
       name="${prefix}tool0">
     </link>
-    <!-- tool0_joint -->
     <joint
       name="${prefix}tool0_joint"
@@ -441,5 +439,5 @@
         link="${prefix}tool0" />
     </joint>
-    <link name="${prefix}elfin_dummy_gripper"/>
+    <!--<link name="${prefix}elfin_dummy_gripper"/>
     <joint name="${prefix}elfin_dummy_joint" type="fixed">
       <origin
@@ -450,5 +448,5 @@
       <child
         link="${prefix}elfin_dummy_gripper" />
-    </joint>
+    </joint>-->
   </xacro:macro>
 </robot>
